File: R3_CH340_Adapter.brd (EAGLE design)
At the start: 68.6 x 53.3 mm, 56 parts, among them IC1 SSW-115-01-G-S-LL, IC2 SSW-115-01-G-S-LL, Q1 BC846, Q2 BC856ALT1SMD, Q3 BC846, Q4 BC856ALT1SMD, U1 AP3012UKTR-E1, U2 AP3012UKTR-E1

Commit message: release v0.3 final design
Parts:
- moved LED3 5.52 mm to (60.8, 12.8)
- moved LED4 5.52 mm to (55.2, 12.8)
Routing:
- net N$8: track 12.6 -> 17.9 mm
- net N$4: track 15.3 -> 13.6 mm
Other:
- board text added: "+12VSRC"
- board text added: "+5VOUT"
- board text added: "+5VSRC"
- board text added: "RESET"

Commit message: v0.3 test OK
Parts:
- R28: value 1K8 -> 470R
