File: R3_CH340_Adapter.sch (EAGLE design)
At the start: 55 parts, among them IC1 SSW-115-01-G-S-LL, IC2 SSW-115-01-G-S-LL, Q1 BC846, Q2 BC856ALT1SMD, Q3 BC846, Q4 BC856ALT1SMD, U1 AP3012UKTR-E1, U2 AP3012UKTR-E1

Commit message: v0.3 test OK
Parts:
- R28: value 1K8 -> 470R
Changed lines of the file:
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@@
 <part name="Q4" library="transistor-pnp" library_urn="urn:adsk.eagle:library:399" deviceset="BC856*" device="SMD" package3d_urn="urn:adsk.eagle:package:28748/2" technology="ALT1"/>
 <part name="GND3" library="supply1" library_urn="urn:adsk.eagle:library:371" deviceset="GND" device=""/>
-<part name="R28" library="rcl" library_urn="urn:adsk.eagle:library:334" deviceset="R-EU_" device="R0805" package3d_urn="urn:adsk.eagle:package:23553/2" value="1K8"/>
+<part name="R28" library="rcl" library_urn="urn:adsk.eagle:library:334" deviceset="R-EU_" device="R0805" package3d_urn="urn:adsk.eagle:package:23553/2" value="470R"/>
 <part name="R30" library="rcl" library_urn="urn:adsk.eagle:library:334" deviceset="R-EU_" device="R0805" package3d_urn="urn:adsk.eagle:package:23553/2" value="4K7"/>
 <part name="LED3" library="led" library_urn="urn:adsk.eagle:library:259" deviceset="LED" device="CHIP-LED0805" package3d_urn="urn:adsk.eagle:package:15818/2" value="YELLOW"/>
